Commit message: Refactor launch file and add RViz configuration; integrate RealSense camera sensors in URDF

File: src/labbot_description/urdf/labbot.xacro (robot description, xacro)
@@ -124,4 +124,11 @@
   </collision>
 </link>
+<!-- Optical frame - required for correct point cloud orientation in RViz -->
+<joint name="realsense_optical_joint" type="fixed">
+  <parent link="realsense_DCAM_1"/>
+  <child  link="realsense_DCAM_1_optical"/>
+  <origin xyz="0 0 0" rpy="1.57 3.14 1.57"/>   <!-- This is the magic rotation -->
+</joint>
+<link name="realsense_DCAM_1_optical"/>
 <joint name="left_wheel_joint" type="continuous">
   <origin xyz="-0.007821 0.134829 0.065288" rpy="0 0 0"/>

Commit message: Add cafe table and ground plane models with SDF configurations
- Created new SDF models for a cafe table and ground plane, including collision and visual elements.
- Added model configuration files for both models with metadata such as name, version, author, and description.
- Updated the package.xml to include a dependency on robot_localization.
- Enhanced setup.py to include new model directories for installation.
- Modified labbot.xacro to include an IMU link and joint.
- Created a new world file for a cafe environment, including multiple instances of the cafe table model.
- Introduced a new labbot_slam package with launch files for RTAB-Map integration and IMU sensor configuration.
- Added necessary files for the labbot_slam package including setup.py, package.xml, and resource files.
- Included a comprehensive Apache License for the labbot_slam package.

File: src/labbot_description/urdf/labbot.xacro (robot description, xacro)
@@ -131,4 +131,10 @@
 </joint>
 <link name="realsense_DCAM_1_optical"/>
+<link name="imu_link"/>
+<joint name="imu_joint" type="fixed">
+  <parent link="base_link"/>
+  <child link="imu_link"/>
+  <origin xyz="0 0 0"/>
+</joint>
 <joint name="left_wheel_joint" type="continuous">
   <origin xyz="-0.007821 0.134829 0.065288" rpy="0 0 0"/>

Commit message: Add navigation and SLAM launch files for labbot
- Created `nav2.launch.py` to set up the Nav2 stack with depth image to laser scan conversion.
- Added `rtabmap_nav2.launch.py` to integrate RTAB-Map with Nav2 for autonomous navigation.
- Updated `package.xml` to include dependencies for Nav2 and depth image processing.
- Modified `setup.py` to install new launch files and configuration files.
- Introduced `rtabmap.launch.py` for RTAB-Map configuration with improved parameter handling.
- Removed obsolete `mapping_rtabmap.launch.py` to streamline launch files.
- Added `rtabmap_slam.launch.py` to manage SLAM operations with RTAB-Map.
- Created RViz configuration file `slam.rviz` for visualizing SLAM data.
-Nav2 working

File: src/labbot_description/urdf/labbot.xacro (robot description, xacro)
@@ -155,4 +155,5 @@
   <axis xyz="0.003611 5.5e-05 0.999993"/>
   <limit upper="1.570796" lower="-1.570796" effort="100" velocity="100"/>
+  <dynamics damping="20.0" friction="10.0"/>
 </joint>
 <joint name="cam_joint" type="revolute">
@@ -162,4 +163,5 @@
   <axis xyz="4e-06 1.0 -5.5e-05"/>
   <limit upper="1.570796" lower="-1.570796" effort="100" velocity="100"/>
+  <dynamics damping="20.0" friction="10.0"/>
 </joint>
 <joint name="camera_joint" type="fixed">
